Commit message: add delay between motors

File: dof6robot_ws/description/ros2_control/dof6robot.ros2_control.xacro (robot description, xacro)
@@ -5,8 +5,9 @@
       <hardware>
         <plugin>dof6robot_control/RobotHardware</plugin>
-        <param name="port_name">/dev/ttyUSB0</param>
+        <param name="usb_port">/dev/ttyUSB0</param>
         <param name="baud_rate">115200</param>
       </hardware>
       <joint name="joint1">
+        <param name="servo_id">0</param>
         <command_interface name="position">
           <param name="min">-1.57</param>
@@ -19,30 +20,32 @@
         <state_interface name="position"/>
         <!-- <state_interface name="velocity"/> -->
-      <param name="servo_id">2</param>
+      <!-- <param name="servo_id">2</param> -->
       </joint>
-      <!-- <joint name="joint2">
+      <joint name="joint2">
+        <param name="servo_id">1</param>
         <command_interface name="position">
+          <param name="min">-1.57</param>
+          <param name="max">1.57</param>
+        </command_interface>
+        <!-- <command_interface name="velocity">
           <param name="min">-1</param>
           <param name="max">1</param>
+        </command_interface> -->
+        <state_interface name="position"/>
+        <!-- <state_interface name="velocity"/> -->
+      </joint>
+      <joint name="joint3">
+        <param name="servo_id">2</param>
+        <command_interface name="position">
+          <param name="min">-1.57</param>
+          <param name="max">1.57</param>
         </command_interface>
-        <command_interface name="velocity">
+        <!-- <command_interface name="velocity">
           <param name="min">-1</param>
           <param name="max">1</param>
-        </command_interface>
+        </command_interface> -->
         <state_interface name="position"/>
-        <state_interface name="velocity"/>
+        <!-- <state_interface name="velocity"/> -->
       </joint>
-      <joint name="joint3">
-        <command_interface name="position">
-          <param name="min">-1</param>
-          <param name="max">1</param>
-        </command_interface>
-        <command_interface name="velocity">
-          <param name="min">-1</param>
-          <param name="max">1</param>
-        </command_interface>
-        <state_interface name="position"/>
-        <state_interface name="velocity"/>
-      </joint> -->
     </ros2_control>
   </xacro:macro>

File: dof6robot_ws/description/urdf/dof6robot.urdf.xacro (robot description, xacro)
@@ -1,76 +1,13 @@
 <?xml version="1.0"?>
 <robot xmlns:xacro="http://www.ros.org/wiki/xacro" name="dof6_robot">
+  <xacro:arg name="enable_joint1" default="true" />
+  <xacro:arg name="enable_joint2" default="true" />
+  <xacro:arg name="enable_joint3" default="true" />
   <!-- Import robot ros2_control description -->
+  <xacro:include filename = "$(find dof6robot_control)/description/dof6robot.description.xacro" />
+  <xacro:robot_description enable_joint1="$(arg enable_joint1)" enable_joint2="$(arg enable_joint2)" enable_joint3="$(arg enable_joint3)" />
+    <!-- Import robot ros2_control description -->
   <xacro:include filename = "$(find dof6robot_control)/ros2_control/dof6robot.ros2_control.xacro" />
-  <link name="base_link">
-    <visual>
-      <geometry>
-        <cylinder length="0.05" radius="0.08"/>
-      </geometry>
-      <material name="gray">
-        <color rgba="0.6 0.6 0.6 1"/>
-      </material>
-    </visual>
-  </link>
-  <!-- Link 1 -->
-  <link name="link1">
-    <visual>
-      <geometry>
-        <cylinder length="0.3" radius="0.04"/>
-      </geometry>
-      <origin xyz="0 0 0.15" rpy="0 0 0"/>
-      <material name="blue">
-        <color rgba="0.2 0.2 0.8 1"/>
-      </material>
-    </visual>
-  </link>
-  <!-- Link 2 -->
-  <!-- <link name="link2">
-    <visual>
-      <geometry>
-        <cylinder length="0.3" radius="0.04"/>
-      </geometry>
-      <origin xyz="0 0 0.15" rpy="0 0 0"/>
-      <material name="green">
-        <color rgba="0.2 0.8 0.2 1"/>
-      </material>
-    </visual>
-  </link> -->
-  <!-- Link 3 -->
-  <!-- <link name="link3">
-    <visual>
-      <geometry>
-        <cylinder length="0.3" radius="0.04"/>
-      </geometry>
-      <origin xyz="0 0 0.15" rpy="0 0 0"/>
-      <material name="red">
-        <color rgba="0.8 0.2 0.2 1"/>
-      </material>
-    </visual>
-  </link> -->
-  <!-- Joint 1: base_link to link1 -->
-  <joint name="joint1" type="revolute">
-    <parent link="base_link"/>
-    <child link="link1"/>
-    <origin xyz="0 0 0.05" rpy="0 0 0"/>
-    <axis xyz="0 0 1"/>
-    <limit lower="-1.57" upper="1.57" effort="10" velocity="2"/>
-  </joint>
-  <!-- Joint 2: link1 to link2 -->
-  <!-- <joint name="joint2" type="revolute">
-    <parent link="link1"/>
-    <child link="link2"/>
-    <origin xyz="0 0 0.3" rpy="0 0 0"/>
-    <axis xyz="0 1 0"/>
-    <limit lower="-1.57" upper="1.57" effort="10" velocity="2"/>
-  </joint> -->
-  <!-- Joint 3: link2 to link3 -->
-  <!-- <joint name="joint3" type="revolute">
-    <parent link="link2"/>
-    <child link="link3"/>
-    <origin xyz="0 0 0.3" rpy="0 0 0"/>
-    <axis xyz="0 1 0"/>
-    <limit lower="-1.57" upper="1.57" effort="10" velocity="2"/>
-  </joint> -->
   <xacro:robot_ros2_control name="robot" />
+  <link name="world"/>
 </robot>
